Commit message: Add tf_prefix

File: my_robot_cell/my_robot_cell_description/urdf/my_robot_cell.urdf.xacro (robot description, xacro)
@@ -3,4 +3,5 @@
   <xacro:include filename="$(find my_robot_cell_description)/urdf/my_robot_cell_macro.xacro"/>
   <xacro:arg name="ur_type" default="ur3e"/>
+  <xacro:arg name="tf_prefix" default=""/>
   <xacro:arg name="joint_limits_parameters_file" default="$(find ur_description)/config/$(arg ur_type)/joint_limits.yaml"/>
   <xacro:arg name="kinematics_parameters_file" default="$(find ur_description)/config/$(arg ur_type)/default_kinematics.yaml"/>
@@ -12,4 +13,5 @@
     parent="world"
     ur_type="$(arg ur_type)"
+    tf_prefix="$(arg tf_prefix)"
     joint_limits_parameters_file="$(arg joint_limits_parameters_file)"
     kinematics_parameters_file="$(arg kinematics_parameters_file)"

File: my_robot_cell/my_robot_cell_description/urdf/my_robot_cell_macro.xacro (robot description, xacro)
@@ -15,4 +15,5 @@
     *origin
     ur_type
+    tf_prefix:=''
     joint_limits_parameters_file
     kinematics_parameters_file
@@ -20,10 +21,10 @@
     visual_parameters_file
     ">
-    <joint name="table_base_joint" type="fixed">
+    <joint name="${tf_prefix}table_base_joint" type="fixed">
       <xacro:insert_block name="origin" />
       <parent link="${parent}" />
-      <child link="table" />
-    </joint>
-    <link name="table">
+      <child link="${tf_prefix}table" />
+    </joint>
+    <link name="${tf_prefix}table">
       <visual>
         <geometry>
@@ -40,8 +41,8 @@
       </collision>
     </link>
-    <link name="robot_mount"/>
-    <joint name="base_to_robot_mount" type="fixed">
-      <parent link="table"/>
-      <child link="robot_mount"/>
+    <link name="${tf_prefix}robot_mount"/>
+    <joint name="${tf_prefix}base_to_robot_mount" type="fixed">
+      <parent link="${tf_prefix}table"/>
+      <child link="${tf_prefix}robot_mount"/>
       <origin xyz="0.40 0.53 0.0" rpy="0 0 ${pi}" />
     </joint>
@@ -49,6 +50,6 @@
     <xacro:ur_robot
       name="${ur_type}"
-      tf_prefix=""
-      parent="robot_mount"
+      tf_prefix="${tf_prefix}"
+      parent="${tf_prefix}robot_mount"
       joint_limits_parameters_file="${joint_limits_parameters_file}"
       kinematics_parameters_file="${kinematics_parameters_file}"
@@ -60,10 +61,10 @@
     </xacro:ur_robot>
     <!-- HAND E -->
-    <joint name="robotiq_hande_coupler_joint" type="fixed">
+    <joint name="${tf_prefix}robotiq_hande_coupler_joint" type="fixed">
       <origin xyz="0 0 0.00695" rpy="0 0 ${-pi/2.0}"/>
-      <parent link="tool0"/>
-      <child link="robotiq_hande_coupler"/>
-    </joint>
-    <link name="robotiq_hande_coupler">
+      <parent link="${tf_prefix}tool0"/>
+      <child link="${tf_prefix}robotiq_hande_coupler"/>
+    </joint>
+    <link name="${tf_prefix}robotiq_hande_coupler">
       <inertial>
         <mass value="0.168"/>
@@ -82,10 +83,10 @@
       </visual>
     </link>
-    <joint name="robotiq_hande_base_joint" type="fixed">
+    <joint name="${tf_prefix}robotiq_hande_base_joint" type="fixed">
       <origin rpy="0 0 0" xyz="0 0 0.055"/>
-      <parent link="robotiq_hande_coupler"/>
-      <child link="robotiq_hande_link"/>
-    </joint>
-    <link name="robotiq_hande_link">
+      <parent link="${tf_prefix}robotiq_hande_coupler"/>
+      <child link="${tf_prefix}robotiq_hande_link"/>
+    </joint>
+    <link name="${tf_prefix}robotiq_hande_link">
       <inertial>
         <mass value="0.86387"/>
@@ -105,12 +106,12 @@
       </visual>
     </link>
-    <joint name="robotiq_hande_left_finger_joint" type="prismatic">
+    <joint name="${tf_prefix}robotiq_hande_left_finger_joint" type="prismatic">
       <origin rpy="0 0 0" xyz="0 -0.025 0.0345"/>
-      <parent link="robotiq_hande_link"/>
-      <child link="robotiq_hande_left_finger"/>
+      <parent link="${tf_prefix}robotiq_hande_link"/>
+      <child link="${tf_prefix}robotiq_hande_left_finger"/>
       <axis xyz="0 1 0"/>
       <limit effort="130" lower="0" upper="0.025" velocity="0.15"/>
     </joint>
-    <link name="robotiq_hande_left_finger">
+    <link name="${tf_prefix}robotiq_hande_left_finger">
       <inertial>
         <origin rpy="0 0 0" xyz="0 0 0"/>
@@ -132,13 +133,13 @@
       </visual>
     </link>
-    <joint name="robotiq_hande_right_finger_joint" type="prismatic">
+    <joint name="${tf_prefix}robotiq_hande_right_finger_joint" type="prismatic">
       <origin rpy="0 0 0" xyz="0 0.025 0.0345"/>
-      <parent link="robotiq_hande_link"/>
-      <child link="robotiq_hande_right_finger"/>
+      <parent link="${tf_prefix}robotiq_hande_link"/>
+      <child link="${tf_prefix}robotiq_hande_right_finger"/>
       <axis xyz="0 -1 0"/>
       <limit effort="130" lower="0" upper="0.025" velocity="0.15"/>
-      <mimic joint="robotiq_hande_left_finger_joint" multiplier="1" offset="0"/>
-    </joint>
-    <link name="robotiq_hande_right_finger">
+      <mimic joint="${tf_prefix}robotiq_hande_left_finger_joint" multiplier="1" offset="0"/>
+    </joint>
+    <link name="${tf_prefix}robotiq_hande_right_finger">
       <inertial>
         <origin rpy="0 0 0" xyz="0 0 0"/>
@@ -160,10 +161,10 @@
       </visual>
     </link>
-    <joint name="robotiq_hande_end_joint" type="fixed">
+    <joint name="${tf_prefix}robotiq_hande_end_joint" type="fixed">
       <origin rpy="0 0 0" xyz="0 0 0.095"/>
-      <parent link="robotiq_hande_link"/>
-      <child link="robotiq_hande_end"/>
-    </joint>
-    <link name="robotiq_hande_end"/>
+      <parent link="${tf_prefix}robotiq_hande_link"/>
+      <child link="${tf_prefix}robotiq_hande_end"/>
+    </joint>
+    <link name="${tf_prefix}robotiq_hande_end"/>
     <!-- Mount -->
     <material name="silver">
@@ -180,5 +181,5 @@
     </material>
     <!-- Mount -->
-    <link name="mount">
+    <link name="${tf_prefix}mount">
       <inertial>
         <origin xyz="0.046989528833305955 -0.025915479612535458 0.02673309777483681" rpy="0 0 0"/>
@@ -202,5 +203,5 @@
     </link>
     <!-- ZED -->
-    <link name="zed2i">
+    <link name="${tf_prefix}zed2i">
       <inertial>
         <origin xyz="-0.014940784453936096 -8.359960537301925e-07 0.004021717834959214" rpy="0 0 0"/>
@@ -222,5 +223,5 @@
       </collision>
     </link>
-    <link name="zed2i_cam_right">
+    <link name="${tf_prefix}zed2i_cam_right">
       <inertial>
         <origin xyz="-3.5072307380534795e-07 9.204312224203592e-08 0.000500234126710776" rpy="0 0 0"/>
@@ -236,5 +237,5 @@
       </visual>
     </link>
-    <link name="zed2i_cam_left">
+    <link name="${tf_prefix}zed2i_cam_left">
       <inertial>
         <origin xyz="-3.507230769139724e-07 9.2043121124874e-08 0.0005002341267107864" rpy="0 0 0"/>
@@ -250,30 +251,30 @@
       </visual>
     </link>
-    <joint name="mount_joint" type="fixed">
+    <joint name="${tf_prefix}mount_joint" type="fixed">
       <origin xyz="0.016 0.027 -0.0314" rpy="1.570796 0 0"/>
-      <parent link="robotiq_hande_link"/>
-      <child link="mount"/>
-    </joint>
-    <joint name="joint_zed_mount" type="fixed">
+      <parent link="${tf_prefix}robotiq_hande_link"/>
+      <child link="${tf_prefix}mount"/>
+    </joint>
+    <joint name="${tf_prefix}joint_zed_mount" type="fixed">
       <origin xyz="0.071152 -0.027 0.023609" rpy="0 0 0"/>
-      <parent link="mount"/>
-      <child link="zed2i"/>
-    </joint>
-    <joint name="joint_zed_right" type="fixed">
+      <parent link="${tf_prefix}mount"/>
+      <child link="${tf_prefix}zed2i"/>
+    </joint>
+    <joint name="${tf_prefix}joint_zed_right" type="fixed">
       <origin xyz="-0.015125 0.06 -0.015495" rpy="0 0 0"/>
-      <parent link="zed2i"/>
-      <child link="zed2i_cam_right"/>
-    </joint>
-    <joint name="joint_zed_left" type="fixed">
+      <parent link="${tf_prefix}zed2i"/>
+      <child link="${tf_prefix}zed2i_cam_right"/>
+    </joint>
+    <joint name="${tf_prefix}joint_zed_left" type="fixed">
       <origin xyz="-0.015125 -0.06 -0.015495" rpy="0 0 0"/>
-      <parent link="zed2i"/>
-      <child link="zed2i_cam_left"/>
-    </joint>
-    <joint name="joint_to_zed_camera_link" type="fixed">
+      <parent link="${tf_prefix}zed2i"/>
+      <child link="${tf_prefix}zed2i_cam_left"/>
+    </joint>
+    <joint name="${tf_prefix}joint_to_zed_camera_link" type="fixed">
       <origin xyz="0 0 0" rpy="0 1.570796327 3.141592654"/>
-      <parent link="zed2i"/>
-      <child link="zed_camera_link"/>
-    </joint>
-    <link name="zed_camera_link"/>
+      <parent link="${tf_prefix}zed2i"/>
+      <child link="${tf_prefix}zed_camera_link"/>
+    </joint>
+    <link name="${tf_prefix}zed_camera_link"/>
   </xacro:macro>
 </robot>
