Commit message: Offset Mount Collison due to bolts

File: my_robot_cell/my_robot_cell_description/urdf/my_robot_cell_macro.xacro (robot description, xacro)
@@ -194,5 +194,6 @@
       </visual>
       <collision>
-        <origin xyz="-0.016 0.0666 0.027" rpy="0 0 0"/>
+        <!-- Offset collision up by 1 cm because of bolt -->
+        <origin xyz="-0.006 0.0666 0.027" rpy="0 0 0"/>
         <geometry>
           <mesh filename="package://my_robot_cell_description/meshes/mount/mount_1.stl" scale="0.001 0.001 0.001"/>

Commit message: Offset Cam mount for safety

File: my_robot_cell/my_robot_cell_description/urdf/my_robot_cell_macro.xacro (robot description, xacro)
@@ -272,5 +272,5 @@
     </joint>
     <joint name="${tf_prefix}joint_to_zed_camera_link" type="fixed">
-      <origin xyz="0 0 0" rpy="0 1.570796327 3.141592654"/>
+      <origin xyz="0 0 -0.018" rpy="0 1.570796327 3.141592654"/>
       <parent link="${tf_prefix}zed2i"/>
       <child link="${tf_prefix}zed_camera_link"/>
